Commit message: modify for ubuntu20.04 and fixed for mobile robot

File: urdf/livox_HAP.xacro (robot description, xacro)
@@ -1,89 +1,91 @@
 <?xml version="1.0"?>
 <robot xmlns:xacro="http://ros.org/wiki/xacro">
-  <xacro:property name="M_PI" value="3.14159"/>
-  <xacro:property name="laser_min_range" value="0.1"/>
-  <xacro:property name="laser_max_range" value="200.0"/>
-  <xacro:property name="ros_topic" value="scan"/>
-  <xacro:property name="samples" value="45300"/>
-  <xacro:property name="downsample" value="1"/>
-  <xacro:macro name="null_inertial">
-    <inertial>
-      <mass value="0.1"/>
-    <inertia ixx="0.01" ixy="0" ixz="0"
-          iyy="0.01" iyz="0"
-          izz="0.01"/>
-    </inertial>
-  </xacro:macro>
-  <xacro:macro name="Livox_Mid_gazebo_sensor" params="visualize:=True update_rate:=10 resolution:=0.002 noise_mean:=0.0 noise_stddev:=0.01 name:=livox">
-    <gazebo reference="${name}">
-      <sensor type="ray" name="laser_${name}">
-        <pose>0 0 0 0 0 0</pose>
-        <visualize>${visualize}</visualize>
-        <update_rate>${update_rate}</update_rate>
-        <!-- This ray plgin is only for visualization. -->
-        <plugin name="gazebo_ros_laser_controller" filename="liblivox_laser_simulation.so">
-			<ray>
-			  <scan>
-				<horizontal>
-				<samples>100</samples>
-				<resolution>1</resolution>
-				<min_angle>${-60/180*M_PI}</min_angle>
-				<max_angle>${60/180*M_PI}</max_angle>
-				</horizontal>
-				<vertical>
-				<samples>50</samples>
-				<resolution>1</resolution>
-				<min_angle>${-12.5/180*M_PI}</min_angle>
-				<max_angle>${12.5/180*M_PI}</max_angle>
-				</vertical>
-			  </scan>
-			  <range>
-				<min>${laser_min_range}</min>
-				<max>${laser_max_range}</max>
-				<resolution>${resolution}</resolution>
-			  </range>
-			  <noise>
-				<type>gaussian</type>
-				<mean>${noise_mean}</mean>
-				<stddev>${noise_stddev}</stddev>
-			  </noise>
-			</ray>
-          <visualize>${visualize}</visualize>
-		  <samples>${samples}</samples>
-		  <downsample>${downsample}</downsample>
-		  <csv_file_name>package://livox_laser_simulation/scan_mode/HAP.csv</csv_file_name>
-		  <ros_topic>${ros_topic}</ros_topic>
-        </plugin>
-      </sensor>
-    </gazebo>
-  </xacro:macro>
-  <xacro:macro name="Livox_Mid40" params="visualize:=True name:=livox">
-    <link name="${name}_base">
-      <xacro:null_inertial/>
-      <visual>
-        <origin xyz="0.00 0 0.0" rpy="0 0 0"/>
-        <geometry>
-          <mesh filename="package://livox_laser_simulation/meshes/livox_mid40.dae">
-          </mesh>
-        </geometry>
-      </visual>
-      <collision>
-		  <origin xyz="0 0 0" rpy="0 0 0" /> <geometry> <mesh
-		  filename="package://livox_laser_simulation/meshes/livox_mid40.dae">
-		  </mesh> </geometry>
-      </collision>
-    </link>
-    <link name="${name}">
-      <xacro:null_inertial/>
-    </link>
-    <joint name="${name}_to_${name}_base_joint" type="fixed">
-      <parent link="${name}_base"/>
-      <child link="${name}"/>
-      <origin rpy="0 0 0" xyz="0.0 0.0 1.6"/>
-    </joint>
-    <xacro:Livox_Mid_gazebo_sensor name="${name}" visualize="${visualize}"/>
-  </xacro:macro>
-    <xacro:Livox_Mid40 name="livox"/>
-  <xacro:include filename="$(find livox_laser_simulation)/urdf/standardrobots_oasis300.xacro"/>
-  <xacro:link_oasis name="oasis"/>
+    <xacro:property name="M_PI" value="3.14159" />
+    <xacro:property name="laser_min_range" value="0.1" />
+    <xacro:property name="laser_max_range" value="200.0" />
+    <xacro:property name="ros_topic" value="scan" />
+    <xacro:property name="samples" value="45300" />
+    <xacro:property name="downsample" value="1" />
+    <xacro:macro name="null_inertial">
+        <inertial>
+            <mass value="0.1" />
+            <inertia ixx="0.01" ixy="0" ixz="0"
+                iyy="0.01" iyz="0"
+                izz="0.01" />
+        </inertial>
+    </xacro:macro>
+    <xacro:macro name="Livox_Mid_gazebo_sensor"
+        params="visualize:=True update_rate:=10 resolution:=0.002 noise_mean:=0.0 noise_stddev:=0.01 name:=livox">
+        <gazebo reference="${name}">
+            <sensor type="ray" name="laser_${name}">
+                <pose>0 0 0 0 0 0</pose>
+                <visualize>${visualize}</visualize>
+                <update_rate>${update_rate}</update_rate>
+                <!-- This ray plgin is only for visualization. -->
+                <plugin name="gazebo_ros_laser_controller" filename="liblivox_laser_simulation.so">
+                    <ray>
+                        <scan>
+                            <horizontal>
+                                <samples>100</samples>
+                                <resolution>1</resolution>
+                                <min_angle>${-60/180*M_PI}</min_angle>
+                                <max_angle>${60/180*M_PI}</max_angle>
+                            </horizontal>
+                            <vertical>
+                                <samples>50</samples>
+                                <resolution>1</resolution>
+                                <min_angle>${-12.5/180*M_PI}</min_angle>
+                                <max_angle>${12.5/180*M_PI}</max_angle>
+                            </vertical>
+                        </scan>
+                        <range>
+                            <min>${laser_min_range}</min>
+                            <max>${laser_max_range}</max>
+                            <resolution>${resolution}</resolution>
+                        </range>
+                        <noise>
+                            <type>gaussian</type>
+                            <mean>${noise_mean}</mean>
+                            <stddev>${noise_stddev}</stddev>
+                        </noise>
+                    </ray>
+                    <visualize>${visualize}</visualize>
+                    <samples>${samples}</samples>
+                    <downsample>${downsample}</downsample>
+                    <csv_file_name>package://livox_laser_simulation/scan_mode/HAP.csv</csv_file_name>
+                    <ros_topic>${ros_topic}</ros_topic>
+                    <frame_name>${name}</frame_name>
+                </plugin>
+            </sensor>
+        </gazebo>
+    </xacro:macro>
+    <xacro:macro name="Livox_Mid40" params="visualize:=True name:=livox">
+        <link name="${name}_base">
+            <xacro:null_inertial />
+            <visual>
+                <origin xyz="0.00 0 0.0" rpy="0 0 0" />
+                <geometry>
+                    <mesh filename="package://livox_laser_simulation/meshes/livox_mid40.dae">
+                    </mesh>
+                </geometry>
+            </visual>
+            <collision>
+                <origin xyz="0 0 0" rpy="0 0 0" />
+                <geometry>
+                    <mesh
+                        filename="package://livox_laser_simulation/meshes/livox_mid40.dae">
+                    </mesh>
+                </geometry>
+            </collision>
+        </link>
+        <link name="${name}">
+            <xacro:null_inertial />
+        </link>
+        <joint name="${name}_to_${name}_base_joint" type="fixed">
+            <parent link="${name}_base" />
+            <child link="${name}" />
+            <origin rpy="0 0 0" xyz="0.0 0.0 1.6" />
+        </joint>
+        <xacro:Livox_Mid_gazebo_sensor name="${name}" visualize="${visualize}" />
+    </xacro:macro>
 </robot>

File: urdf/livox_avia.xacro (robot description, xacro)
@@ -1,93 +1,97 @@
 <?xml version="1.0"?>
 <robot xmlns:xacro="http://ros.org/wiki/xacro">
-  <xacro:property name="M_PI" value="3.14159"/>
-  <xacro:property name="laser_min_range" value="0.1"/>
-  <xacro:property name="laser_max_range" value="200.0"/>
-  <xacro:property name="horizontal_fov" value="70.4"/>
-  <xacro:property name="vertical_fov" value="77.2"/>
-  <xacro:property name="ros_topic" value="scan"/>
-  <xacro:property name="samples" value="24000"/>
-  <xacro:property name="downsample" value="1"/>
-  <xacro:macro name="null_inertial">
-    <inertial>
-      <mass value="0.1"/>
-    <inertia ixx="0.01" ixy="0" ixz="0"
-          iyy="0.01" iyz="0"
-          izz="0.01"/>
-    </inertial>
-  </xacro:macro>
-  <xacro:macro name="Livox_Mid_gazebo_sensor" params="visualize:=True update_rate:=10 resolution:=0.002 noise_mean:=0.0 noise_stddev:=0.01 name:=livox">
-    <gazebo reference="${name}">
-      <sensor type="ray" name="laser_${name}">
-        <pose>0 0 0 0 0 0</pose>
-        <visualize>${visualize}</visualize>
-        <update_rate>${update_rate}</update_rate>
-        <!-- This ray plgin is only for visualization. -->
-        <plugin name="gazebo_ros_laser_controller" filename="liblivox_laser_simulation.so">
-			<ray>
-			  <scan>
-				<horizontal>
-				<samples>100</samples>
-				<resolution>1</resolution>
-				<min_angle>${-horizontal_fov/360*M_PI}</min_angle>
-				<max_angle>${horizontal_fov/360*M_PI}</max_angle>
-				</horizontal>
-				<vertical>
-				<samples>50</samples>
-				<resolution>1</resolution>
-				<min_angle>${-vertical_fov/360*M_PI}</min_angle>
-				<max_angle>${vertical_fov/360*M_PI}</max_angle>
-				</vertical>
-			  </scan>
-			  <range>
-				<min>${laser_min_range}</min>
-				<max>${laser_max_range}</max>
-				<resolution>${resolution}</resolution>
-			  </range>
-			  <noise>
-				<type>gaussian</type>
-				<mean>${noise_mean}</mean>
-				<stddev>${noise_stddev}</stddev>
-			  </noise>
-			</ray>
-          <visualize>${visualize}</visualize>
-		  <samples>${samples}</samples>
-		  <downsample>${downsample}</downsample>
-		  <csv_file_name>package://livox_laser_simulation/scan_mode/avia.csv</csv_file_name>
-		  <ros_topic>${ros_topic}</ros_topic>
-        </plugin>
-      </sensor>
-    </gazebo>
-  </xacro:macro>
-  <xacro:macro name="Livox_AVIA" params="visualize:=True name:=livox">
-    <link name="${name}_base">
-      <xacro:null_inertial/>
-      <visual>
-        <origin xyz="0.00 0 0.00" rpy="0 0 0"/>
-        <geometry>
-          <mesh filename="package://livox_laser_simulation/meshes/livox_mid40.dae">
-          </mesh>
-        </geometry>
-      </visual>
-      <collision>
-          <origin xyz="0 0 0" rpy="0 0 0" />
-          <geometry>
-          <mesh filename="package://livox_laser_simulation/meshes/livox_mid40.dae">
-          </mesh>
-          </geometry>
-      </collision>
-    </link>
-    <link name="${name}">
-      <xacro:null_inertial/>
-    </link>
-    <joint name="${name}_to_${name}_base_joint" type="fixed">
-      <parent link="${name}_base"/>
-      <child link="${name}"/>
-      <origin rpy="0 0 0" xyz="0.0 0.0 0.0"/>
-    </joint>
-    <xacro:Livox_Mid_gazebo_sensor name="${name}" visualize="${visualize}"/>
-  </xacro:macro>
-    <xacro:Livox_AVIA name="livox"/>
-  <xacro:include filename="$(find livox_laser_simulation)/urdf/standardrobots_oasis300.xacro"/>
-  <xacro:link_oasis name="oasis"/>
+    <xacro:property name="M_PI" value="3.14159" />
+    <xacro:property name="laser_min_range" value="0.1" />
+    <xacro:property name="laser_max_range" value="200.0" />
+    <xacro:property name="horizontal_fov" value="70.4" />
+    <xacro:property name="vertical_fov" value="77.2" />
+    <xacro:property name="ros_topic" value="scan" />
+    <xacro:property name="samples" value="24000" />
+    <xacro:property name="downsample" value="1" />
+    <xacro:macro name="null_inertial">
+        <inertial>
+            <mass value="0.1" />
+            <inertia ixx="0.01" ixy="0" ixz="0"
+                iyy="0.01" iyz="0"
+                izz="0.01" />
+        </inertial>
+    </xacro:macro>
+    <xacro:macro name="Livox_Mid_gazebo_sensor"
+        params="visualize:=True update_rate:=10 resolution:=0.002 noise_mean:=0.0 noise_stddev:=0.01 name:=livox">
+        <gazebo reference="${name}">
+            <sensor type="ray" name="laser_${name}">
+                <pose>0 0 0 0 0 0</pose>
+                <visualize>${visualize}</visualize>
+                <update_rate>${update_rate}</update_rate>
+                <!-- This ray plgin is only for visualization. -->
+                <plugin name="gazebo_ros_laser_controller" filename="liblivox_laser_simulation.so">
+                    <ray>
+                        <scan>
+                            <horizontal>
+                                <samples>100</samples>
+                                <resolution>1</resolution>
+                                <min_angle>${-horizontal_fov/360*M_PI}</min_angle>
+                                <max_angle>${horizontal_fov/360*M_PI}</max_angle>
+                            </horizontal>
+                            <vertical>
+                                <samples>50</samples>
+                                <resolution>1</resolution>
+                                <min_angle>${-vertical_fov/360*M_PI}</min_angle>
+                                <max_angle>${vertical_fov/360*M_PI}</max_angle>
+                            </vertical>
+                        </scan>
+                        <range>
+                            <min>${laser_min_range}</min>
+                            <max>${laser_max_range}</max>
+                            <resolution>${resolution}</resolution>
+                        </range>
+                        <noise>
+                            <type>gaussian</type>
+                            <mean>${noise_mean}</mean>
+                            <stddev>${noise_stddev}</stddev>
+                        </noise>
+                    </ray>
+                    <visualize>${visualize}</visualize>
+                    <samples>${samples}</samples>
+                    <downsample>${downsample}</downsample>
+                    <csv_file_name>package://livox_laser_simulation/scan_mode/avia.csv</csv_file_name>
+                    <ros_topic>${ros_topic}</ros_topic>
+                    <frame_name>${name}</frame_name>
+                </plugin>
+            </sensor>
+        </gazebo>
+    </xacro:macro>
+    <xacro:macro name="Livox_AVIA" params="visualize:=True name:=livox parent:=base_link">
+        <link name="${name}_base">
+            <xacro:null_inertial />
+            <visual>
+                <origin xyz="0.00 0 0.00" rpy="0 0 0" />
+                <geometry>
+                    <mesh filename="package://livox_laser_simulation/meshes/livox_mid40.dae">
+                    </mesh>
+                </geometry>
+            </visual>
+            <collision>
+                <origin xyz="0 0 0" rpy="0 0 0" />
+                <geometry>
+                    <mesh filename="package://livox_laser_simulation/meshes/livox_mid40.dae">
+                    </mesh>
+                </geometry>
+            </collision>
+        </link>
+        <link name="${name}">
+            <xacro:null_inertial />
+        </link>
+        <joint name="${name}_to_${name}_base_joint" type="fixed">
+            <parent link="${name}_base" />
+            <child link="${name}" />
+            <origin rpy="0 0 0" xyz="0.0 0.0 0.0" />
+        </joint>
+        <joint name="${name}_base_to_parent_joint" type="fixed">
+            <parent link="${parent}" />
+            <child link="${name}_base" />
+            <origin rpy="0 0 0" xyz="0.05 0.0 0.0" />
+        </joint>
+        <xacro:Livox_Mid_gazebo_sensor name="${name}" visualize="${visualize}" />
+    </xacro:macro>
 </robot>

File: urdf/livox_horizon.xacro (robot description, xacro)
@@ -56,4 +56,5 @@
 		  <csv_file_name>package://livox_laser_simulation/scan_mode/horizon.csv</csv_file_name>
 		  <ros_topic>${ros_topic}</ros_topic>
+          <frame_name>${name}</frame_name>
         </plugin>
       </sensor>
@@ -86,6 +87,3 @@
     <xacro:Livox_Mid_gazebo_sensor name="${name}" visualize="${visualize}"/>
   </xacro:macro>
-    <xacro:Livox_HORIZON name="livox"/>
-  <xacro:include filename="$(find livox_laser_simulation)/urdf/standardrobots_oasis300.xacro"/>
-  <xacro:link_oasis name="oasis"/>
 </robot>

File: urdf/livox_mid360.xacro (robot description, xacro)
@@ -54,4 +54,5 @@
 		  <csv_file_name>package://livox_laser_simulation/scan_mode/mid360.csv</csv_file_name>
 		  <ros_topic>${ros_topic}</ros_topic>
+          <frame_name>${name}</frame_name>
         </plugin>
       </sensor>
@@ -84,6 +85,3 @@
     <xacro:Livox_Mid_gazebo_sensor name="${name}" visualize="${visualize}"/>
   </xacro:macro>
-    <xacro:Livox_Mid40 name="livox"/>
-  <xacro:include filename="$(find livox_laser_simulation)/urdf/standardrobots_oasis300.xacro"/>
-  <xacro:link_oasis name="oasis"/>
 </robot>

File: urdf/livox_mid40.xacro (robot description, xacro)
@@ -56,4 +56,5 @@
 		  <csv_file_name>package://livox_laser_simulation/scan_mode/mid40.csv</csv_file_name>
 		  <ros_topic>${ros_topic}</ros_topic>
+          <frame_name>${name}</frame_name>
         </plugin>
       </sensor>
@@ -86,6 +87,3 @@
     <xacro:Livox_Mid_gazebo_sensor name="${name}" visualize="${visualize}"/>
   </xacro:macro>
-    <xacro:Livox_Mid40 name="livox"/>
-  <xacro:include filename="$(find livox_laser_simulation)/urdf/standardrobots_oasis300.xacro"/>
-  <xacro:link_oasis name="oasis"/>
 </robot>

File: urdf/livox_mid70.xacro (robot description, xacro)
@@ -56,4 +56,5 @@
 		  <csv_file_name>package://livox_laser_simulation/scan_mode/mid70.csv</csv_file_name>
 		  <ros_topic>${ros_topic}</ros_topic>
+          <frame_name>${name}</frame_name>
         </plugin>
       </sensor>
@@ -88,6 +89,3 @@
     <xacro:Livox_Mid_gazebo_sensor name="${name}" visualize="${visualize}"/>
   </xacro:macro>
-    <xacro:Livox_Mid70 name="livox"/>
-  <xacro:include filename="$(find livox_laser_simulation)/urdf/standardrobots_oasis300.xacro"/>
-  <xacro:link_oasis name="oasis"/>
 </robot>

File: urdf/livox_tele.xacro (robot description, xacro)
@@ -56,4 +56,5 @@
 		  <csv_file_name>package://livox_laser_simulation/scan_mode/tele.csv</csv_file_name>
 		  <ros_topic>${ros_topic}</ros_topic>
+          <frame_name>${name}</frame_name>
         </plugin>
       </sensor>
@@ -88,6 +89,3 @@
     <xacro:Livox_Mid_gazebo_sensor name="${name}" visualize="${visualize}"/>
   </xacro:macro>
-    <xacro:Livox_TELE name="livox"/>
-  <xacro:include filename="$(find livox_laser_simulation)/urdf/standardrobots_oasis300.xacro"/>
-  <xacro:link_oasis name="oasis"/>
 </robot>

File: urdf/standardrobots_oasis300.xacro (robot description, xacro)
@@ -3,18 +3,19 @@
     <!-- Defining the colors used in this robot -->
     <material name="Black">
-        <color rgba="0 0 0 1"/>
+        <color rgba="0 0 0 1" />
     </material>
     <material name="White">
-        <color rgba="1 1 1 1"/>
+        <color rgba="1 1 1 1" />
     </material>
     <material name="Blue">
-        <color rgba="0 0 1 1"/>
+        <color rgba="0 0 1 1" />
     </material>
     <material name="Red">
-        <color rgba="1 0 0 1"/>
+        <color rgba="1 0 0 1" />
     </material>
-	<!-- Constants --> <xacro:property name="M_PI" value="3.14159"/>
-	<!-- inertial matrix -->
-	<xacro:macro name="inertial_matrix" params="mass">
+    <!-- Constants -->
+    <xacro:property name="M_PI" value="3.14159" />
+    <!-- inertial matrix -->
+    <xacro:macro name="inertial_matrix" params="mass">
         <inertial>
             <mass value="${mass}" />
@@ -22,41 +23,44 @@
         </inertial>
     </xacro:macro>
-<!--
+    <!--
     world link is named as "link"
 -->
-	<xacro:macro name="link_oasis" params="name:=oasis base_link:=oasis_300 world_link:=link">
-    <link name="link"/>
-    <!-- base_link -->
-    <link name="oasis_300">
-        <visual>
-			<origin xyz="0.00 0 0.05" rpy="0 0 0"/>
-            <geometry>
-				  <mesh filename="package://livox_laser_simulation/meshes/standardrobots.STL"/>
-            </geometry>
-        </visual>
-        <collision>
-			<origin xyz="0.00 0 0.05" rpy="0 0 0"/>
-            <geometry>
-				  <mesh filename="package://livox_laser_simulation/meshes/standardrobots.STL"/>
-            </geometry>
-        </collision>
-        <xacro:inertial_matrix mass="1"/>
-		<kinematic>1</kinematic>
-		<gravity>9.8</gravity>
-    </link>
-    <gazebo reference="oasis_300">
-        <material>Gazebo/White</material>
-    </gazebo>
-	<joint name="fixed" type="fixed">
-		<parent link="${world_link}"/>
-		<child link="${base_link}"/>
-		<origin xyz="0.0 0 0.05" rpy="0 0 ${M_PI/2}" />
-	</joint>
-	<joint name="livox_base_joint" type="fixed">
-        <parent link="${base_link}"/>
-        <child link="livox_base"/>
-        <origin rpy="0 0 1.5707"
-                xyz="0.0 0.4 0.3057"/>
-    </joint>
+    <xacro:macro name="link_oasis" params="name:=oasis base_link:=oasis_300 world_link:=link">
+        <link name="link" />
+        <!-- base_link -->
+        <link name="oasis_300">
+            <visual>
+                <origin xyz="0.00 0 0.05" rpy="0 0 0" />
+                <geometry>
+                    <mesh filename="package://livox_laser_simulation/meshes/standardrobots.STL" />
+                </geometry>
+            </visual>
+            <collision>
+                <origin xyz="0.00 0 0.05" rpy="0 0 0" />
+                <geometry>
+                    <mesh filename="package://livox_laser_simulation/meshes/standardrobots.STL" />
+                </geometry>
+            </collision>
+            <xacro:inertial_matrix mass="1" />
+            <kinematic>1</kinematic>
+            <gravity>9.8</gravity>
+        </link>
+        <gazebo reference="oasis_300">
+            <material>Gazebo/White</material>
+        </gazebo>
+        <joint name="fixed" type="fixed">
+            <parent link="${world_link}" />
+            <child link="${base_link}" />
+            <origin xyz="0.0 0 0.05" rpy="0 0 ${M_PI/2}" />
+        </joint>
+        <joint name="livox_base_joint" type="fixed">
+            <parent link="${base_link}" />
+            <child link="livox_base" />
+            <origin rpy="0 0 1.5707"
+                xyz="0.0 0.4 0.3057" />
+        </joint>
     </xacro:macro>
+    <xacro:include filename="$(find livox_laser_simulation)/urdf/livox_mid40.xacro"/>
+    <xacro:Livox_Mid40 name="livox" />
+    <xacro:link_oasis name="oasis" />
 </robot>
