Commit message: add support for livox laser

File: urdf/livox_HAP.xacro (robot description, xacro)
@@ -60,5 +60,5 @@
         </gazebo>
     </xacro:macro>
-    <xacro:macro name="Livox_Mid40" params="visualize:=True name:=livox">
+    <xacro:macro name="Livox_Mid40" params="visualize:=True name:=livox parent:=base_link">
         <link name="${name}_base">
             <xacro:null_inertial />
@@ -87,4 +87,9 @@
             <origin rpy="0 0 0" xyz="0.0 0.0 1.6" />
         </joint>
+        <joint name="${name}_base_to_parent_joint" type="fixed">
+            <parent link="${parent}" />
+            <child link="${name}_base" />
+            <origin rpy="0 0 0" xyz="0.05 0.0 0.0" />
+        </joint>
         <xacro:Livox_Mid_gazebo_sensor name="${name}" visualize="${visualize}" />
     </xacro:macro>

File: urdf/livox_horizon.xacro (robot description, xacro)
@@ -61,5 +61,5 @@
     </gazebo>
   </xacro:macro>
-  <xacro:macro name="Livox_HORIZON" params="visualize:=True name:=livox">
+  <xacro:macro name="Livox_HORIZON" params="visualize:=True name:=livox parent:=base_link">
     <link name="${name}_base">
       <xacro:null_inertial/>
@@ -85,4 +85,9 @@
       <origin rpy="0 0 0" xyz="0.0 0.0 0.0"/>
     </joint>
+    <joint name="${name}_base_to_parent_joint" type="fixed">
+        <parent link="${parent}" />
+        <child link="${name}_base" />
+        <origin rpy="0 0 0" xyz="0.05 0.0 0.0" />
+    </joint>
     <xacro:Livox_Mid_gazebo_sensor name="${name}" visualize="${visualize}"/>
   </xacro:macro>

File: urdf/livox_mid360.xacro (robot description, xacro)
@@ -59,5 +59,5 @@
     </gazebo>
   </xacro:macro>
-  <xacro:macro name="Livox_Mid40" params="visualize:=True name:=livox">
+  <xacro:macro name="Livox_Mid40" params="visualize:=True name:=livox parent:=base_link">
     <link name="${name}_base">
       <xacro:null_inertial/>
@@ -83,4 +83,9 @@
       <origin rpy="0 0 0" xyz="0.0 1.0 0.2"/>
     </joint>
+    <joint name="${name}_base_to_parent_joint" type="fixed">
+        <parent link="${parent}" />
+        <child link="${name}_base" />
+        <origin rpy="0 0 0" xyz="0.05 0.0 0.0" />
+    </joint>
     <xacro:Livox_Mid_gazebo_sensor name="${name}" visualize="${visualize}"/>
   </xacro:macro>

File: urdf/livox_mid40.xacro (robot description, xacro)
@@ -61,5 +61,5 @@
     </gazebo>
   </xacro:macro>
-  <xacro:macro name="Livox_Mid40" params="visualize:=True name:=livox">
+  <xacro:macro name="Livox_Mid40" params="visualize:=True name:=livox parent:=base_link">
     <link name="${name}_base">
       <xacro:null_inertial/>
@@ -85,4 +85,9 @@
       <origin rpy="0 0 0" xyz="0.0 0.0 0.0"/>
     </joint>
+    <joint name="${name}_base_to_parent_joint" type="fixed">
+        <parent link="${parent}" />
+        <child link="${name}_base" />
+        <origin rpy="0 0 0" xyz="0.05 0.0 0.0" />
+    </joint>
     <xacro:Livox_Mid_gazebo_sensor name="${name}" visualize="${visualize}"/>
   </xacro:macro>

File: urdf/livox_mid70.xacro (robot description, xacro)
@@ -61,5 +61,5 @@
     </gazebo>
   </xacro:macro>
-  <xacro:macro name="Livox_Mid70" params="visualize:=True name:=livox">
+  <xacro:macro name="Livox_Mid70" params="visualize:=True name:=livox parent:=base_link">
     <link name="${name}_base">
       <xacro:null_inertial/>
@@ -87,4 +87,9 @@
       <origin rpy="0 0 0" xyz="0.0 0.0 0.0"/>
     </joint>
+    <joint name="${name}_base_to_parent_joint" type="fixed">
+        <parent link="${parent}" />
+        <child link="${name}_base" />
+        <origin rpy="0 0 0" xyz="0.05 0.0 0.0" />
+    </joint>
     <xacro:Livox_Mid_gazebo_sensor name="${name}" visualize="${visualize}"/>
   </xacro:macro>

File: urdf/livox_tele.xacro (robot description, xacro)
@@ -61,5 +61,5 @@
     </gazebo>
   </xacro:macro>
-  <xacro:macro name="Livox_TELE" params="visualize:=True name:=livox">
+  <xacro:macro name="Livox_TELE" params="visualize:=True name:=livox parent:=base_link">
     <link name="${name}_base">
       <xacro:null_inertial/>
@@ -87,4 +87,9 @@
       <origin rpy="0 0 0" xyz="0.0 0.0 0.0"/>
     </joint>
+    <joint name="${name}_base_to_parent_joint" type="fixed">
+        <parent link="${parent}" />
+        <child link="${name}_base" />
+        <origin rpy="0 0 0" xyz="0.05 0.0 0.0" />
+    </joint>
     <xacro:Livox_Mid_gazebo_sensor name="${name}" visualize="${visualize}"/>
   </xacro:macro>
