Commit message: add options for choosing lidar msg type and fix the bug including the ignition/math.hh header file

File: urdf/livox_avia.xacro (robot description, xacro)
@@ -4,63 +4,16 @@
     <xacro:property name="laser_min_range" value="0.1" />
     <xacro:property name="laser_max_range" value="200.0" />
+    <!-- 水平FOV，度为单位 -->
     <xacro:property name="horizontal_fov" value="70.4" />
-    <xacro:property name="vertical_fov" value="77.2" />
+    <!-- 垂直上下限角，度为单位 -->
+    <xacro:property name="min_vertical_angle" value="-${77.2/2}" />
+    <xacro:property name="max_vertical_angle" value="${77.2/2}" />
     <xacro:property name="ros_topic" value="scan" />
     <xacro:property name="samples" value="24000" />
     <xacro:property name="downsample" value="1" />
-    <xacro:macro name="null_inertial">
-        <inertial>
-            <mass value="0.1" />
-            <inertia ixx="0.01" ixy="0" ixz="0"
-                iyy="0.01" iyz="0"
-                izz="0.01" />
-        </inertial>
-    </xacro:macro>
-    <xacro:macro name="Livox_Mid_gazebo_sensor"
-        params="visualize:=True update_rate:=10 resolution:=0.002 noise_mean:=0.0 noise_stddev:=0.01 name:=livox">
-        <gazebo reference="${name}">
-            <sensor type="ray" name="laser_${name}">
-                <pose>0 0 0 0 0 0</pose>
-                <visualize>${visualize}</visualize>
-                <update_rate>${update_rate}</update_rate>
-                <!-- This ray plgin is only for visualization. -->
-                <plugin name="gazebo_ros_laser_controller" filename="liblivox_laser_simulation.so">
-                    <ray>
-                        <scan>
-                            <horizontal>
-                                <samples>100</samples>
-                                <resolution>1</resolution>
-                                <min_angle>${-horizontal_fov/360*M_PI}</min_angle>
-                                <max_angle>${horizontal_fov/360*M_PI}</max_angle>
-                            </horizontal>
-                            <vertical>
-                                <samples>50</samples>
-                                <resolution>1</resolution>
-                                <min_angle>${-vertical_fov/360*M_PI}</min_angle>
-                                <max_angle>${vertical_fov/360*M_PI}</max_angle>
-                            </vertical>
-                        </scan>
-                        <range>
-                            <min>${laser_min_range}</min>
-                            <max>${laser_max_range}</max>
-                            <resolution>${resolution}</resolution>
-                        </range>
-                        <noise>
-                            <type>gaussian</type>
-                            <mean>${noise_mean}</mean>
-                            <stddev>${noise_stddev}</stddev>
-                        </noise>
-                    </ray>
-                    <visualize>${visualize}</visualize>
-                    <samples>${samples}</samples>
-                    <downsample>${downsample}</downsample>
-                    <csv_file_name>package://livox_laser_simulation/scan_mode/avia.csv</csv_file_name>
-                    <ros_topic>${ros_topic}</ros_topic>
-                    <frame_name>${name}</frame_name>
-                </plugin>
-            </sensor>
-        </gazebo>
-    </xacro:macro>
-    <xacro:macro name="Livox_AVIA" params="visualize:=True name:=livox parent:=base_link">
+    <xacro:property name="publish_pointcloud_type" value="1"/>
+    <xacro:property name="csv_file_name" value="package://livox_laser_simulation/scan_mode/avia.csv"/>
+    <xacro:include filename="$(find livox_laser_simulation)/urdf/livox_gazebo_sensor.xacro"/>
+    <xacro:macro name="Livox_Avia" params="visualize:=True name:=livox parent:=base_link">
         <link name="${name}_base">
             <xacro:null_inertial />
@@ -93,5 +46,5 @@
             <origin rpy="0 0 0" xyz="0.0 0.0 0.0" />
         </joint>
-        <xacro:Livox_Mid_gazebo_sensor name="${name}" visualize="${visualize}" />
+        <xacro:Livox_gazebo_sensor name="${name}" visualize="${visualize}" publish_pointcloud_type="${publish_pointcloud_type}" />
     </xacro:macro>
 </robot>

File: urdf/livox_hap.xacro (robot description, xacro)
@@ -5,28 +5,29 @@
     <xacro:property name="laser_max_range" value="200.0" />
     <!-- 水平FOV，度为单位 -->
-    <xacro:property name="horizontal_fov" value="38.4" />
+    <xacro:property name="horizontal_fov" value="120" />
     <!-- 垂直上下限角，度为单位 -->
-    <xacro:property name="min_vertical_angle" value="-${38.4/2}" />
-    <xacro:property name="max_vertical_angle" value="${38.4/2}" />
+    <xacro:property name="min_vertical_angle" value="-${25.0/2}" />
+    <xacro:property name="max_vertical_angle" value="${25.0/2}" />
     <xacro:property name="ros_topic" value="scan" />
-    <xacro:property name="samples" value="10000"/>
+    <xacro:property name="samples" value="45300" />
     <xacro:property name="downsample" value="1" />
     <xacro:property name="publish_pointcloud_type" value="1"/>
-    <xacro:property name="csv_file_name" value="package://livox_laser_simulation/scan_mode/mid40.csv"/>
+    <xacro:property name="csv_file_name" value="package://livox_laser_simulation/scan_mode/HAP.csv"/>
     <xacro:include filename="$(find livox_laser_simulation)/urdf/livox_gazebo_sensor.xacro"/>
-    <xacro:macro name="Livox_Mid40" params="visualize:=True name:=livox parent:=base_link publish_pointcloud_type:=1" >
+    <xacro:macro name="Livox_Hap" params="visualize:=True name:=livox parent:=base_link">
         <link name="${name}_base">
             <xacro:null_inertial />
             <visual>
-                <origin xyz="0.045 0 0.04" rpy="0 0 0" />
+                <origin xyz="0.00 0 0.0" rpy="0 0 0" />
                 <geometry>
-                    <mesh filename="package://livox_laser_simulation/meshes/livox_mid40.dae">
+                    <mesh filename="package://livox_laser_simulation/meshes/livox_HAP.dae">
                     </mesh>
                 </geometry>
             </visual>
             <collision>
-                <origin xyz="0.045 0 0.04" rpy="0 0 0" />
+                <origin xyz="0 0 0" rpy="0 0 0" />
                 <geometry>
-                    <mesh filename="package://livox_laser_simulation/meshes/livox_mid40.dae">
+                    <mesh
+                        filename="package://livox_laser_simulation/meshes/livox_HAP.dae">
                     </mesh>
                 </geometry>
@@ -39,5 +40,5 @@
             <parent link="${name}_base" />
             <child link="${name}" />
-            <origin rpy="0 0 0" xyz="0.0 0.0 0.04" />
+            <origin rpy="0 0 0" xyz="0.0 0.0 0.0" />
         </joint>
         <joint name="${name}_base_to_parent_joint" type="fixed">

File: urdf/livox_horizon.xacro (robot description, xacro)
@@ -4,63 +4,16 @@
     <xacro:property name="laser_min_range" value="0.1" />
     <xacro:property name="laser_max_range" value="200.0" />
+    <!-- 水平FOV，度为单位 -->
     <xacro:property name="horizontal_fov" value="81.7" />
-    <xacro:property name="vertical_fov" value="25.1" />
+    <!-- 垂直上下限角，度为单位 -->
+    <xacro:property name="min_vertical_angle" value="-${25.1/2}" />
+    <xacro:property name="max_vertical_angle" value="${25.1/2}" />
     <xacro:property name="ros_topic" value="scan" />
     <xacro:property name="samples" value="24000" />
     <xacro:property name="downsample" value="1" />
-    <xacro:macro name="null_inertial">
-        <inertial>
-            <mass value="0.1" />
-            <inertia ixx="0.01" ixy="0" ixz="0"
-                iyy="0.01" iyz="0"
-                izz="0.01" />
-        </inertial>
-    </xacro:macro>
-    <xacro:macro name="Livox_Mid_gazebo_sensor"
-        params="visualize:=True update_rate:=10 resolution:=0.002 noise_mean:=0.0 noise_stddev:=0.01 name:=livox">
-        <gazebo reference="${name}">
-            <sensor type="ray" name="laser_${name}">
-                <pose>0 0 0 0 0 0</pose>
-                <visualize>${visualize}</visualize>
-                <update_rate>${update_rate}</update_rate>
-                <!-- This ray plgin is only for visualization. -->
-                <plugin name="gazebo_ros_laser_controller" filename="liblivox_laser_simulation.so">
-                    <ray>
-                        <scan>
-                            <horizontal>
-                                <samples>100</samples>
-                                <resolution>1</resolution>
-                                <min_angle>${-horizontal_fov/360*M_PI}</min_angle>
-                                <max_angle>${horizontal_fov/360*M_PI}</max_angle>
-                            </horizontal>
-                            <vertical>
-                                <samples>50</samples>
-                                <resolution>1</resolution>
-                                <min_angle>${-vertical_fov/360*M_PI}</min_angle>
-                                <max_angle>${vertical_fov/360*M_PI}</max_angle>
-                            </vertical>
-                        </scan>
-                        <range>
-                            <min>${laser_min_range}</min>
-                            <max>${laser_max_range}</max>
-                            <resolution>${resolution}</resolution>
-                        </range>
-                        <noise>
-                            <type>gaussian</type>
-                            <mean>${noise_mean}</mean>
-                            <stddev>${noise_stddev}</stddev>
-                        </noise>
-                    </ray>
-                    <visualize>${visualize}</visualize>
-                    <samples>${samples}</samples>
-                    <downsample>${downsample}</downsample>
-                    <csv_file_name>package://livox_laser_simulation/scan_mode/horizon.csv</csv_file_name>
-                    <ros_topic>${ros_topic}</ros_topic>
-                    <frame_name>${name}</frame_name>
-                </plugin>
-            </sensor>
-        </gazebo>
-    </xacro:macro>
-    <xacro:macro name="Livox_HORIZON" params="visualize:=True name:=livox parent:=base_link">
+    <xacro:property name="publish_pointcloud_type" value="1"/>
+    <xacro:property name="csv_file_name" value="package://livox_laser_simulation/scan_mode/horizon.csv"/>
+    <xacro:include filename="$(find livox_laser_simulation)/urdf/livox_gazebo_sensor.xacro"/>
+    <xacro:macro name="Livox_Horizon" params="visualize:=True name:=livox parent:=base_link">
         <link name="${name}_base">
             <xacro:null_inertial />
@@ -93,5 +46,5 @@
             <origin rpy="0 0 0" xyz="0.0 0.0 0.0" />
         </joint>
-        <xacro:Livox_Mid_gazebo_sensor name="${name}" visualize="${visualize}" />
+        <xacro:Livox_gazebo_sensor name="${name}" visualize="${visualize}" publish_pointcloud_type="${publish_pointcloud_type}" />
     </xacro:macro>
 </robot>

File: urdf/livox_mid360.xacro (robot description, xacro)
@@ -7,4 +7,5 @@
     <xacro:property name="samples" value="24000" />
     <xacro:property name="downsample" value="1" />
+    <xacro:property name="publish_pointcloud_type" value="1"/>
     <xacro:macro name="null_inertial">
         <inertial>
@@ -15,5 +16,5 @@
         </inertial>
     </xacro:macro>
-    <xacro:macro name="Livox_Mid_gazebo_sensor"
+    <xacro:macro name="Livox_gazebo_sensor"
         params="visualize:=True update_rate:=10 resolution:=0.002 noise_mean:=0.0 noise_stddev:=0.01 name:=livox">
         <gazebo reference="${name}">
@@ -55,4 +56,5 @@
                     <csv_file_name>package://livox_laser_simulation/scan_mode/mid360.csv</csv_file_name>
                     <ros_topic>${ros_topic}</ros_topic>
+                    <publish_pointcloud_type>${publish_pointcloud_type}</publish_pointcloud_type>
                     <frame_name>${name}</frame_name>
                 </plugin>
@@ -60,5 +62,5 @@
         </gazebo>
     </xacro:macro>
-    <xacro:macro name="Livox_Mid40" params="visualize:=True name:=livox parent:=base_link">
+    <xacro:macro name="Livox_Mid360" params="visualize:=True name:=livox parent:=base_link">
         <link name="${name}_base">
             <xacro:null_inertial />
@@ -92,5 +94,5 @@
             <origin rpy="0 0 0" xyz="0.0 0.0 0.0" />
         </joint>
-        <xacro:Livox_Mid_gazebo_sensor name="${name}" visualize="${visualize}" />
+        <xacro:Livox_gazebo_sensor name="${name}" visualize="${visualize}" />
     </xacro:macro>
 </robot>

File: urdf/livox_mid70.xacro (robot description, xacro)
@@ -4,62 +4,15 @@
     <xacro:property name="laser_min_range" value="0.1" />
     <xacro:property name="laser_max_range" value="200.0" />
+    <!-- 水平FOV，度为单位 -->
     <xacro:property name="horizontal_fov" value="70.4" />
-    <xacro:property name="vertical_fov" value="70.4" />
+    <!-- 垂直上下限角，度为单位 -->
+    <xacro:property name="min_vertical_angle" value="-${70.4/2}" />
+    <xacro:property name="max_vertical_angle" value="${70.4/2}" />
     <xacro:property name="ros_topic" value="scan" />
     <xacro:property name="samples" value="10000" />
     <xacro:property name="downsample" value="1" />
-    <xacro:macro name="null_inertial">
-        <inertial>
-            <mass value="0.1" />
-            <inertia ixx="0.01" ixy="0" ixz="0"
-                iyy="0.01" iyz="0"
-                izz="0.01" />
-        </inertial>
-    </xacro:macro>
-    <xacro:macro name="Livox_Mid_gazebo_sensor"
-        params="visualize:=True update_rate:=10 resolution:=0.002 noise_mean:=0.0 noise_stddev:=0.01 name:=livox">
-        <gazebo reference="${name}">
-            <sensor type="ray" name="laser_${name}">
-                <pose>0 0 0 0 0 0</pose>
-                <visualize>${visualize}</visualize>
-                <update_rate>${update_rate}</update_rate>
-                <!-- This ray plgin is only for visualization. -->
-                <plugin name="gazebo_ros_laser_controller" filename="liblivox_laser_simulation.so">
-                    <ray>
-                        <scan>
-                            <horizontal>
-                                <samples>100</samples>
-                                <resolution>1</resolution>
-                                <min_angle>${-horizontal_fov/360*M_PI}</min_angle>
-                                <max_angle>${horizontal_fov/360*M_PI}</max_angle>
-                            </horizontal>
-                            <vertical>
-                                <samples>50</samples>
-                                <resolution>1</resolution>
-                                <min_angle>${-vertical_fov/360*M_PI}</min_angle>
-                                <max_angle>${vertical_fov/360*M_PI}</max_angle>
-                            </vertical>
-                        </scan>
-                        <range>
-                            <min>${laser_min_range}</min>
-                            <max>${laser_max_range}</max>
-                            <resolution>${resolution}</resolution>
-                        </range>
-                        <noise>
-                            <type>gaussian</type>
-                            <mean>${noise_mean}</mean>
-                            <stddev>${noise_stddev}</stddev>
-                        </noise>
-                    </ray>
-                    <visualize>${visualize}</visualize>
-                    <samples>${samples}</samples>
-                    <downsample>${downsample}</downsample>
-                    <csv_file_name>package://livox_laser_simulation/scan_mode/mid70.csv</csv_file_name>
-                    <ros_topic>${ros_topic}</ros_topic>
-                    <frame_name>${name}</frame_name>
-                </plugin>
-            </sensor>
-        </gazebo>
-    </xacro:macro>
+    <xacro:property name="publish_pointcloud_type" value="1"/>
+    <xacro:property name="csv_file_name" value="package://livox_laser_simulation/scan_mode/mid70.csv"/>
+    <xacro:include filename="$(find livox_laser_simulation)/urdf/livox_gazebo_sensor.xacro"/>
     <xacro:macro name="Livox_Mid70" params="visualize:=True name:=livox parent:=base_link">
         <link name="${name}_base">
@@ -93,5 +46,5 @@
             <origin rpy="0 0 0" xyz="0.0 0.0 0.0" />
         </joint>
-        <xacro:Livox_Mid_gazebo_sensor name="${name}" visualize="${visualize}" />
+        <xacro:Livox_gazebo_sensor name="${name}" visualize="${visualize}" publish_pointcloud_type="${publish_pointcloud_type}"/>
     </xacro:macro>
 </robot>

File: urdf/livox_tele.xacro (robot description, xacro)
@@ -4,63 +4,16 @@
     <xacro:property name="laser_min_range" value="0.1" />
     <xacro:property name="laser_max_range" value="200.0" />
+    <!-- 水平FOV，度为单位 -->
     <xacro:property name="horizontal_fov" value="14.5" />
-    <xacro:property name="vertical_fov" value="16.1" />
+    <!-- 垂直上下限角，度为单位 -->
+    <xacro:property name="min_vertical_angle" value="-${16.1/2}" />
+    <xacro:property name="max_vertical_angle" value="${16.1/2}" />
     <xacro:property name="ros_topic" value="scan" />
     <xacro:property name="samples" value="24000" />
     <xacro:property name="downsample" value="1" />
-    <xacro:macro name="null_inertial">
-        <inertial>
-            <mass value="0.1" />
-            <inertia ixx="0.01" ixy="0" ixz="0"
-                iyy="0.01" iyz="0"
-                izz="0.01" />
-        </inertial>
-    </xacro:macro>
-    <xacro:macro name="Livox_Mid_gazebo_sensor"
-        params="visualize:=True update_rate:=10 resolution:=0.002 noise_mean:=0.0 noise_stddev:=0.01 name:=livox">
-        <gazebo reference="${name}">
-            <sensor type="ray" name="laser_${name}">
-                <pose>0 0 0 0 0 0</pose>
-                <visualize>${visualize}</visualize>
-                <update_rate>${update_rate}</update_rate>
-                <!-- This ray plgin is only for visualization. -->
-                <plugin name="gazebo_ros_laser_controller" filename="liblivox_laser_simulation.so">
-                    <ray>
-                        <scan>
-                            <horizontal>
-                                <samples>100</samples>
-                                <resolution>1</resolution>
-                                <min_angle>${-horizontal_fov/360*M_PI}</min_angle>
-                                <max_angle>${horizontal_fov/360*M_PI}</max_angle>
-                            </horizontal>
-                            <vertical>
-                                <samples>50</samples>
-                                <resolution>1</resolution>
-                                <min_angle>${-vertical_fov/360*M_PI}</min_angle>
-                                <max_angle>${vertical_fov/360*M_PI}</max_angle>
-                            </vertical>
-                        </scan>
-                        <range>
-                            <min>${laser_min_range}</min>
-                            <max>${laser_max_range}</max>
-                            <resolution>${resolution}</resolution>
-                        </range>
-                        <noise>
-                            <type>gaussian</type>
-                            <mean>${noise_mean}</mean>
-                            <stddev>${noise_stddev}</stddev>
-                        </noise>
-                    </ray>
-                    <visualize>${visualize}</visualize>
-                    <samples>${samples}</samples>
-                    <downsample>${downsample}</downsample>
-                    <csv_file_name>package://livox_laser_simulation/scan_mode/tele.csv</csv_file_name>
-                    <ros_topic>${ros_topic}</ros_topic>
-                    <frame_name>${name}</frame_name>
-                </plugin>
-            </sensor>
-        </gazebo>
-    </xacro:macro>
-    <xacro:macro name="Livox_TELE" params="visualize:=True name:=livox parent:=base_link">
+    <xacro:property name="publish_pointcloud_type" value="1"/>
+    <xacro:property name="csv_file_name" value="package://livox_laser_simulation/scan_mode/tele.csv"/>
+    <xacro:include filename="$(find livox_laser_simulation)/urdf/livox_gazebo_sensor.xacro"/>
+    <xacro:macro name="Livox_Tele" params="visualize:=True name:=livox parent:=base_link">
         <link name="${name}_base">
             <xacro:null_inertial />
@@ -93,5 +46,5 @@
             <origin rpy="0 0 0" xyz="0.0 0.0 0.0" />
         </joint>
-        <xacro:Livox_Mid_gazebo_sensor name="${name}" visualize="${visualize}" />
+        <xacro:Livox_gazebo_sensor name="${name}" visualize="${visualize}" publish_pointcloud_type="${publish_pointcloud_type}" />
     </xacro:macro>
 </robot>
