Commit message: modify the conversion from angle to radian in xacro

File: urdf/livox_avia.xacro (robot description, xacro)
@@ -1,5 +1,4 @@
 <?xml version="1.0"?>
 <robot xmlns:xacro="http://ros.org/wiki/xacro">
-    <xacro:property name="M_PI" value="3.14159" />
     <xacro:property name="laser_min_range" value="0.1" />
     <xacro:property name="laser_max_range" value="200.0" />

File: urdf/livox_gazebo_sensor.xacro (robot description, xacro)
@@ -23,12 +23,12 @@
                                 <samples>100</samples>
                                 <resolution>1</resolution>
-                                <min_angle>${-horizontal_fov/360.0*M_PI}</min_angle>
-                                <max_angle>${horizontal_fov/360.0*M_PI}</max_angle>
+                                <min_angle>${radians(-horizontal_fov/2.0)}</min_angle>
+                                <max_angle>${radians(horizontal_fov/2.0)}</max_angle>
                             </horizontal>
                             <vertical>
                                 <samples>50</samples>
                                 <resolution>1</resolution>
-                                <min_angle>${min_vertical_angle/180.0*M_PI}</min_angle>
-                                <max_angle>${max_vertical_angle/180.0*M_PI}</max_angle>
+                                <min_angle>${radians(min_vertical_angle)}</min_angle>
+                                <max_angle>${radians(max_vertical_angle)}</max_angle>
                             </vertical>
                         </scan>

File: urdf/livox_hap.xacro (robot description, xacro)
@@ -1,5 +1,4 @@
 <?xml version="1.0"?>
 <robot xmlns:xacro="http://ros.org/wiki/xacro">
-    <xacro:property name="M_PI" value="3.14159" />
     <xacro:property name="laser_min_range" value="0.1" />
     <xacro:property name="laser_max_range" value="200.0" />

File: urdf/livox_horizon.xacro (robot description, xacro)
@@ -1,5 +1,4 @@
 <?xml version="1.0"?>
 <robot xmlns:xacro="http://ros.org/wiki/xacro">
-    <xacro:property name="M_PI" value="3.14159" />
     <xacro:property name="laser_min_range" value="0.1" />
     <xacro:property name="laser_max_range" value="200.0" />

File: urdf/livox_mid360.xacro (robot description, xacro)
@@ -1,5 +1,4 @@
 <?xml version="1.0"?>
 <robot xmlns:xacro="http://ros.org/wiki/xacro">
-    <xacro:property name="M_PI" value="3.14159" />
     <xacro:property name="laser_min_range" value="0.1" />
     <xacro:property name="laser_max_range" value="200.0" />
@@ -31,11 +30,11 @@
                                 <resolution>1</resolution>
                                 <min_angle>${0}</min_angle>
-                                <max_angle>${2*M_PI}</max_angle>
+                                <max_angle>${radians(360)}</max_angle>
                             </horizontal>
                             <vertical>
                                 <samples>360</samples>
                                 <resolution>1</resolution>
-                                <min_angle>${-7.22/180*M_PI}</min_angle>
-                                <max_angle>${55.22/180*M_PI}</max_angle>
+                                <min_angle>${radians(-7.22)}</min_angle>
+                                <max_angle>${radians(55.22)}</max_angle>
                             </vertical>
                         </scan>

File: urdf/livox_mid40.xacro (robot description, xacro)
@@ -1,5 +1,4 @@
 <?xml version="1.0"?>
 <robot xmlns:xacro="http://ros.org/wiki/xacro">
-    <xacro:property name="M_PI" value="3.14159" />
     <xacro:property name="laser_min_range" value="0.1" />
     <xacro:property name="laser_max_range" value="200.0" />

File: urdf/livox_mid70.xacro (robot description, xacro)
@@ -1,5 +1,4 @@
 <?xml version="1.0"?>
 <robot xmlns:xacro="http://ros.org/wiki/xacro">
-    <xacro:property name="M_PI" value="3.14159" />
     <xacro:property name="laser_min_range" value="0.1" />
     <xacro:property name="laser_max_range" value="200.0" />

File: urdf/livox_tele.xacro (robot description, xacro)
@@ -1,5 +1,4 @@
 <?xml version="1.0"?>
 <robot xmlns:xacro="http://ros.org/wiki/xacro">
-    <xacro:property name="M_PI" value="3.14159" />
     <xacro:property name="laser_min_range" value="0.1" />
     <xacro:property name="laser_max_range" value="200.0" />

File: urdf/standardrobots_oasis300.xacro (robot description, xacro)
@@ -14,6 +14,4 @@
         <color rgba="1 0 0 1" />
     </material>
-    <!-- Constants -->
-    <xacro:property name="M_PI" value="3.14159" />
     <!-- inertial matrix -->
     <xacro:macro name="inertial_matrix" params="mass">
@@ -52,5 +50,5 @@
             <parent link="${world_link}" />
             <child link="${base_link}" />
-            <origin xyz="0.0 0 0.05" rpy="0 0 ${M_PI/2}" />
+            <origin xyz="0.0 0 0.05" rpy="0 0 ${radians(90)}" />
         </joint>
         <joint name="livox_base_joint" type="fixed">
